File: blind_spot_KICAD/blind_spot_KICAD.kicad_sch (KiCad schematic)
At the start: 0 parts

Commit message: Actualizar esquematico KiCad
Parts:
- added BZ1: Buzzer, symbol Device:Buzzer
- added D2: LED, LED_THT:LED_D5.0mm, symbol Device:LED
- added ESP32_C1, ESP32_C2: ESP32-C3_SUPERMINI_TH, customSimbols:MODULE_ESP32-C3_SUPERMINI_TH, symbol customSimbols:ESP32-C3_SUPERMINI_TH
- added HCSR04: ~, customSimbols:XCVR_HC-SR04, symbol customSimbols:HC_SR04
- added J1, J3: Bateria, Connector_PinHeader_2.54mm:PinHeader_1x02_P2.54mm_Vertical, symbol Connector:Conn_01x02_Pin
- added J2: QTR5000, symbol Connector_Generic:Conn_01x04
- added M1: Motor_DC, symbol Motor:Motor_DC
- added Q1: BC547, Package_TO_SOT_THT:TO-92_Inline, symbol Transistor_BJT:BC547
- added R1: 220, Resistor_THT:R_Axial_DIN0207_L6.3mm_D2.5mm_P10.16mm_Horizontal, symbol Device:R
- added R2: 1k, Resistor_THT:R_Axial_DIN0207_L6.3mm_D2.5mm_P10.16mm_Horizontal, symbol Device:R
- added R3: 10k, Resistor_THT:R_Axial_DIN0207_L6.3mm_D2.5mm_P10.16mm_Horizontal, symbol Device:R
- added R4: LDR03, OptoDevice:R_LDR_10x8.5mm_P7.6mm_Vertical, symbol Sensor_Optical:LDR03
- added R5: 2k2, Resistor_THT:R_Axial_DIN0207_L6.3mm_D2.5mm_P10.16mm_Horizontal, symbol Device:R
- added SW2: SW_MEC_5E, Button_Switch_THT:SW_TH_Tactile_Omron_B3F-10xx, symbol Switch:SW_MEC_5E
Connections:
- new net: D2.1 (K), R1.1
- new net: M1.1 (+), Q1.3 (E)
- new net 3V3: ESP32_C1.3.3 (3V3), ESP32_C2.3.3 (3V3), J2.1 (Pin_1), R4.1
- new net Buzzer: BZ1.1 (+), ESP32_C2.4 (GPIO4)
- new net Echo: ESP32_C2.21 (GPIO21), HCSR04.3 (Echo), R2.1, R5.1
- new net GND: BZ1.2 (-), ESP32_C1.G (GND), ESP32_C2.G (GND), HCSR04.4 (GND), J1.2 (Pin_2), J2.2 (Pin_2), J3.2 (Pin_2), M1.2 (-), R1.2, R3.2, R5.2, SW2.1
- new net LDR: ESP32_C2.1 (GPIO1), R3.1, R4.2
- new net LED1: D2.2 (A), ESP32_C2.5 (GPIO5)
- new net M1: ESP32_C1.10 (GPIO10), Q1.2 (B)
- new net S1: ESP32_C2.0 (GPIO0), J2.4 (Pin_4)
- new net SW1: ESP32_C1.3 (GPIO3), SW2.2
- new net Triger: ESP32_C2.20 (GPIO20), HCSR04.2 (Trigger)
- new net VBat: ESP32_C1.5V, ESP32_C2.5V, HCSR04.1 (VCC), J1.1 (Pin_1), J3.1 (Pin_1), Q1.1 (C), R2.2
Other:
- note added: "BASTON"
- note added: "MUÑECA"
